Commit message: cassie standing

File: robot_descriptions/cassie_description/urdf/cassie_collide.urdf (robot description, URDF)
Before this commit: robot cassie, 18 links, 17 joints
Joints:
- joint ankle_joint_left: limit lower=0.872 upper=2.97 effort=0 velocity=100 -> lower=0.872 upper=2.97 effort=12.2 velocity=100
- joint ankle_joint_right: limit lower=0.872 upper=2.97 effort=0 velocity=100 -> lower=0.872 upper=2.97 effort=12.2 velocity=100
- joint knee_to_shin_left: limit lower=-0.349 upper=0.349 effort=0 velocity=100 -> lower=-0.349 upper=0.349 effort=12.2 velocity=100
- joint knee_to_shin_right: limit lower=-0.349 upper=0.349 effort=0 velocity=100 -> lower=-0.349 upper=0.349 effort=12.2 velocity=100
